File: Pardo.kicad_pcb (KiCad board)
At the start: 2 copper layers, 50.8 x 22.9 mm, 42 parts, among them J1 USB_OTG, J2 Conn_02x01, J3 Conn_02x01, J4 Conn_02x01, J5 Conn_02x01, J7 Conn_02x01, SW1 SW_Push, U1 ATSAMD21G18A-AUT, U2 TPS73733DCQR, U3 MCP73832T-2ACI_OT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

Commit message: Adding more bias
Signed-off-by: Ricardo Mena C <rgacort12@gmail.com>
Routing:
- net GND: vias 13 -> 77
Changed lines of the file:
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@@
     (thickness 1.6)
     (drawings 73)
-    (tracks 510)
+    (tracks 576)
     (zones 0)
     (modules 42)
@@
   )
   (setup
-    (last_trace_width 0.2032)
+    (last_trace_width 0.25)
+    (user_trace_width 0.25)
     (trace_clearance 0.15)
     (zone_clearance 0.254)
@@
   (gr_line (start 126.6571 81.7499) (end 172.4787 81.7499) (layer Edge.Cuts) (width 0.15))
   (gr_line (start 124.2187 102.1715) (end 124.2187 84.2811) (layer Edge.Cuts) (width 0.15))
+  (via (at 154.3558 84.8741) (size 0.4) (drill 0.2) (layers F.Cu B.Cu) (net 2))
   (segment (start 149.1869 93.8075) (end 148.837672 94.156728) (width 0.2032) (layer F.Cu) (net 1))
   (segment (start 149.1869 91.1987) (end 149.1869 93.8075) (width 0.2032) (layer F.Cu) (net 1))
@@
   (segment (start 134.278172 98.5266) (end 134.278172 99.535092) (width 0.3032) (layer F.Cu) (net 2))
   (segment (start 133.6548 98.5266) (end 134.278172 98.5266) (width 0.3032) (layer F.Cu) (net 2))
-  (via (at 155.1305 89.4207) (size 0.6) (drill 0.3937) (layers F.Cu B.Cu) (net 2) (status 1000000))
+  (via (at 155.1305 89.4207) (size 0.6) (drill 0.3937) (layers F.Cu B.Cu) (net 2))
   (via (at 158.772838 91.667989) (size 0.6) (drill 0.3937) (layers F.Cu B.Cu) (net 2))
   (segment (start 158.839727 91.6011) (end 158.772838 91.667989) (width 0.3032) (layer F.Cu) (net 2))
@@
   (via (at 149.2631 100.9523) (size 0.4) (drill 0.2032) (layers F.Cu B.Cu) (net 2))
   (via (at 148.7551 96.5835) (size 0.6) (drill 0.3937) (layers F.Cu B.Cu) (net 2))
+  (via (at 153.5938 84.6201) (size 0.4) (drill 0.2) (layers F.Cu B.Cu) (net 2))
+  (via (at 155.6512 84.9757) (size 0.4) (drill 0.2) (layers F.Cu B.Cu) (net 2))
+  (via (at 151.5618 86.3727) (size 0.4) (drill 0.2) (layers F.Cu B.Cu) (net 2))
+  (via (at 150.7744 87.8205) (size 0.6) (drill 0.3937) (layers F.Cu B.Cu) (net 2))
+  (via (at 149.6822 90.1065) (size 0.6) (drill 0.3937) (layers F.Cu B.Cu) (net 2))
+  (via (at 162.7378 86.6521) (size 0.6) (drill 0.3937) (layers F.Cu B.Cu) (net 2))
+  (via (at 165.2778 86.6521) (size 0.6) (drill 0.3937) (layers F.Cu B.Cu) (net 2))
+  (via (at 165.2778 88.1761) (size 0.6) (drill 0.3937) (layers F.Cu B.Cu) (net 2))
+  (via (at 162.7378 88.1761) (size 0.6) (drill 0.3937) (layers F.Cu B.Cu) (net 2))
+  (via (at 164.0078 87.4141) (size 0.6) (drill 0.3937) (layers F.Cu B.Cu) (net 2))
+  (via (at 164.0078 89.1921) (size 0.6) (drill 0.3937) (layers F.Cu B.Cu) (net 2))
+  (via (at 167.5638 86.6521) (size 0.6) (drill 0.3937) (layers F.Cu B.Cu) (net 2))
+  (via (at 169.5958 85.1281) (size 0.6) (drill 0.3937) (layers F.Cu B.Cu) (net 2))
+  (via (at 165.2778 92.4941) (size 0.6) (drill 0.3937) (layers F.Cu B.Cu) (net 2))
+  (via (at 167.5638 92.4941) (size 0.6) (drill 0.3937) (layers F.Cu B.Cu) (net 2))
+  (via (at 167.5638 90.4621) (size 0.6) (drill 0.3937) (layers F.Cu B.Cu) (net 2))
+  (via (at 167.5638 94.7801) (size 0.6) (drill 0.3937) (layers F.Cu B.Cu) (net 2))
+  (via (at 165.2778 94.7801) (size 0.6) (drill 0.3937) (layers F.Cu B.Cu) (net 2))
+  (via (at 167.5638 97.3201) (size 0.6) (drill 0.3937) (layers F.Cu B.Cu) (net 2))
+  (via (at 167.5638 99.8601) (size 0.6) (drill 0.3937) (layers F.Cu B.Cu) (net 2))
+  (via (at 169.8498 101.1301) (size 0.6) (drill 0.3937) (layers F.Cu B.Cu) (net 2))
+  (via (at 161.2138 95.7961) (size 0.6) (drill 0.3937) (layers F.Cu B.Cu) (net 2))
+  (via (at 155.8798 90.9701) (size 0.6) (drill 0.3937) (layers F.Cu B.Cu) (net 2))
+  (via (at 156.1338 89.4461) (size 0.6) (drill 0.3937) (layers F.Cu B.Cu) (net 2))
+  (via (at 146.4818 96.8121) (size 0.6) (drill 0.3937) (layers F.Cu B.Cu) (net 2))
+  (segment (start 145.0467 96.2159) (end 145.0467 96.2159) (width 0.3032) (layer F.Cu) (net 2))
+  (via (at 145.0467 96.2159) (size 0.6) (drill 0.3937) (layers F.Cu B.Cu) (net 2))
+  (via (at 138.8618 94.7801) (size 0.6) (drill 0.3937) (layers F.Cu B.Cu) (net 2))
+  (via (at 134.7978 95.7961) (size 0.4) (drill 0.2) (layers F.Cu B.Cu) (net 2))
+  (via (at 132.2578 96.0501) (size 0.4) (drill 0.2) (layers F.Cu B.Cu) (net 2))
+  (via (at 129.9718 101.6381) (size 0.6) (drill 0.3937) (layers F.Cu B.Cu) (net 2))
+  (via (at 138.0998 101.6381) (size 0.6) (drill 0.3937) (layers F.Cu B.Cu) (net 2))
+  (via (at 140.1318 101.6381) (size 0.6) (drill 0.3937) (layers F.Cu B.Cu) (net 2))
+  (via (at 154.8638 101.6381) (size 0.6) (drill 0.3937) (layers F.Cu B.Cu) (net 2))
+  (via (at 156.1338 100.3681) (size 0.6) (drill 0.3937) (layers F.Cu B.Cu) (net 2))
+  (via (at 156.1338 101.6381) (size 0.6) (drill 0.3937) (layers F.Cu B.Cu) (net 2))
+  (via (at 161.7218 101.3841) (size 0.6) (drill 0.3937) (layers F.Cu B.Cu) (net 2))
+  (via (at 133.5278 83.0961) (size 0.6) (drill 0.3937) (layers F.Cu B.Cu) (net 2))
+  (via (at 133.5278 84.3661) (size 0.6) (drill 0.3937) (layers F.Cu B.Cu) (net 2))
+  (via (at 133.5278 85.6361) (size 0.6) (drill 0.3937) (layers F.Cu B.Cu) (net 2))
+  (via (at 136.0678 85.6361) (size 0.6) (drill 0.3937) (layers F.Cu B.Cu) (net 2))
+  (via (at 136.0678 84.3661) (size 0.6) (drill 0.3937) (layers F.Cu B.Cu) (net 2))
+  (via (at 136.0678 83.0961) (size 0.6) (drill 0.3937) (layers F.Cu B.Cu) (net 2))
+  (via (at 134.7978 83.6041) (size 0.6) (drill 0.3937) (layers F.Cu B.Cu) (net 2))
+  (via (at 134.7978 84.8741) (size 0.6) (drill 0.3937) (layers F.Cu B.Cu) (net 2))
+  (via (at 137.3378 87.9221) (size 0.6) (drill 0.3937) (layers F.Cu B.Cu) (net 2))
+  (via (at 138.8618 87.9221) (size 0.6) (drill 0.3937) (layers F.Cu B.Cu) (net 2))
+  (via (at 137.3378 89.7001) (size 0.6) (drill 0.3937) (layers F.Cu B.Cu) (net 2))
+  (via (at 132.6388 93.8911) (size 0.6) (drill 0.3937) (layers F.Cu B.Cu) (net 2))
+  (via (at 131.3688 93.8911) (size 0.6) (drill 0.3937) (layers F.Cu B.Cu) (net 2))
+  (via (at 125.1458 93.8911) (size 0.6) (drill 0.3937) (layers F.Cu B.Cu) (net 2))
+  (via (at 126.4158 93.8911) (size 0.6) (drill 0.3937) (layers F.Cu B.Cu) (net 2))
+  (via (at 131.8768 88.0491) (size 0.6) (drill 0.3937) (layers F.Cu B.Cu) (net 2))
+  (via (at 131.8768 90.3351) (size 0.6) (drill 0.3937) (layers F.Cu B.Cu) (net 2))
+  (via (at 129.5908 89.7001) (size 0.6) (drill 0.3937) (layers F.Cu B.Cu) (net 2))
+  (via (at 129.7178 85.6361) (size 0.6) (drill 0.3937) (layers F.Cu B.Cu) (net 2))
+  (via (at 138.4808 98.8441) (size 0.6) (drill 0.3937) (layers F.Cu B.Cu) (net 2))
+  (via (at 139.6238 98.8441) (size 0.6) (drill 0.3937) (layers F.Cu B.Cu) (net 2))
+  (via (at 162.9918 85.3821) (size 0.6) (drill 0.3937) (layers F.Cu B.Cu) (net 2))
+  (via (at 165.1508 85.3821) (size 0.6) (drill 0.3937) (layers F.Cu B.Cu) (net 2))
+  (via (at 165.9128 84.6201) (size 0.6) (drill 0.3937) (layers F.Cu B.Cu) (net 2))
+  (via (at 160.3248 85.2551) (size 0.4) (drill 0.2) (layers F.Cu B.Cu) (net 2))
+  (via (at 143.4338 101.7651) (size 0.4) (drill 0.2) (layers F.Cu B.Cu) (net 2))
+  (via (at 146.2786 102.06482) (size 0.4) (drill 0.2) (layers F.Cu B.Cu) (net 2))
   (segment (start 153.1639 97.9551) (end 153.4687 98.2599) (width 0.2032) (layer F.Cu) (net 3))
   (segment (start 153.4727 98.2559) (end 153.4687 98.2599) (width 0.2032) (layer F.Cu) (net 3))
@@
   (segment (start 155.4861 87.4627) (end 155.4727 87.4761) (width 0.2032) (layer F.Cu) (net 21))
   (segment (start 155.4861 86.0933) (end 155.4861 87.4627) (width 0.2032) (layer F.Cu) (net 21))
-  (segment (start 168.6647 83.0239) (end 166.1541 85.5345) (width 0.2032) (layer F.Cu) (net 22))
-  (via (at 160.4645 85.5345) (size 0.4) (drill 0.2032) (layers F.Cu B.Cu) (net 22))
-  (segment (start 166.1541 85.5345) (end 160.4645 85.5345) (width 0.2032) (layer F.Cu) (net 22))
-  (segment (start 160.040236 85.5345) (end 159.354436 86.2203) (width 0.2032) (layer B.Cu) (net 22))
-  (segment (start 160.4645 85.5345) (end 160.040236 85.5345) (width 0.2032) (layer B.Cu) (net 22))
-  (segment (start 159.354436 86.2203) (end 156.3243 86.2203) (width 0.2032) (layer B.Cu) (net 22))
   (via (at 156.3243 86.2203) (size 0.4) (drill 0.2032) (layers F.Cu B.Cu) (net 22))
   (segment (start 155.9727 86.5719) (end 155.9727 87.4761) (width 0.2032) (layer F.Cu) (net 22))
   (segment (start 156.3243 86.2203) (end 155.9727 86.5719) (width 0.2032) (layer F.Cu) (net 22))
+  (via (at 160.4518 86.0171) (size 0.4) (drill 0.2032) (layers F.Cu B.Cu) (net 22))
+  (segment (start 156.3243 86.2203) (end 156.5275 86.0171) (width 0.2032) (layer B.Cu) (net 22))
+  (segment (start 165.6715 86.0171) (end 160.734642 86.0171) (width 0.2032) (layer F.Cu) (net 22))
+  (segment (start 156.5275 86.0171) (end 160.168958 86.0171) (width 0.2032) (layer B.Cu) (net 22))
+  (segment (start 168.6647 83.0239) (end 165.6715 86.0171) (width 0.2032) (layer F.Cu) (net 22))
+  (segment (start 160.168958 86.0171) (end 160.4518 86.0171) (width 0.2032) (layer B.Cu) (net 22))
+  (segment (start 160.734642 86.0171) (end 160.4518 86.0171) (width 0.2032) (layer F.Cu) (net 22))
   (segment (start 128.7267 92.1847) (end 130.1415 92.1847) (width 0.3032) (layer F.Cu) (net 23))
   (segment (start 130.4675 91.8587) (end 131.5847 91.8587) (width 0.3032) (layer F.Cu) (net 23))

Commit message: minor updates
Signed-off-by: Ricardo Mena C <rgacort12@gmail.com>
Other:
- board text added: "."
Changed lines of the file:
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@@
   (general
     (thickness 1.6)
-    (drawings 73)
+    (drawings 74)
     (tracks 576)
     (zones 0)
@@
   )
   (setup
-    (last_trace_width 0.25)
+    (last_trace_width 0.2032)
     (user_trace_width 0.25)
     (trace_clearance 0.15)
@@
     (pad 1 np_thru_hole circle (at 0 0 90) (size 2.2 2.2) (drill 2.2) (layers *.Cu *.Mask))
   )
+  (gr_text . (at 152.1206 94.7293) (layer F.SilkS)
+    (effects (font (size 1.5 1.5) (thickness 0.3)))
+  )
   (gr_text +3V (at 170.6245 101.4095 90) (layer B.SilkS)
     (effects (font (size 0.8 0.8) (thickness 0.15)) (justify mirror))
@@
   (gr_line (start 126.6571 81.7499) (end 172.4787 81.7499) (layer Edge.Cuts) (width 0.15))
   (gr_line (start 124.2187 102.1715) (end 124.2187 84.2811) (layer Edge.Cuts) (width 0.15))
-  (via (at 154.3558 84.8741) (size 0.4) (drill 0.2) (layers F.Cu B.Cu) (net 2))
   (segment (start 149.1869 93.8075) (end 148.837672 94.156728) (width 0.2032) (layer F.Cu) (net 1))
   (segment (start 149.1869 91.1987) (end 149.1869 93.8075) (width 0.2032) (layer F.Cu) (net 1))
@@
   (segment (start 151.17519 91.6011) (end 150.56959 90.9955) (width 0.2032) (layer F.Cu) (net 1))
   (segment (start 149.3901 90.9955) (end 149.1869 91.1987) (width 0.2032) (layer F.Cu) (net 1))
+  (via (at 154.3558 84.8741) (size 0.4) (drill 0.2) (layers F.Cu B.Cu) (net 2))
   (segment (start 143.5107 97.7519) (end 145.0467 96.2159) (width 0.3032) (layer F.Cu) (net 2))
   (segment (start 142.7107 97.7519) (end 143.5107 97.7519) (width 0.3032) (layer F.Cu) (net 2))
